File: Astable Multivibrator/Astable Multivibrator.kicad_sch (KiCad schematic)
At the start: 11 parts, among them J1 Conn_01x02, Q1 BC547, Q2 BC547

Commit message: feat: Replaced the pin header by a terminal block.
Parts:
- J1: footprint XS:Connector-Breakaway-Header-2.54x0.66mm-2 -> XS:Connector-Wurth-Terminal-Block-2P-3.5mm-691214110002
Changed lines of the file:
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@@
       (effects (font (size 1.27 1.27)) (justify left) hide)
     )
-    (property "Footprint" "XS:Connector-Breakaway-Header-2.54x0.66mm-2" (at 157.48 59.69 0)
+    (property "Footprint" "XS:Connector-Wurth-Terminal-Block-2P-3.5mm-691214110002" (at 157.48 59.69 0)
       (effects (font (size 1.27 1.27)) hide)
     )
